Commit message: change max unmoved steps config

File: envs/isaac_assets/urdf/cube.urdf (robot description, URDF)
Before this commit: robot object, 1 links, 0 joints
Links:
- link object: geometry collision box size=0.16 0.04 0.04; visual box size=0.16 0.04 0.04

Commit message: add handover ezpolicy and change block mass

File: envs/isaac_assets/urdf/cube.urdf (robot description, URDF)
Before this commit: robot object, 1 links, 0 joints
Links:
- link object: mass 0.5 -> 0.1
